File: KiCad/brake control module/brake control module old.kicad_pcb (KiCad board)
At the start: 4 copper layers, 102.5 x 204.2 mm, 280 parts, among them J1 PENDANT ESTOP + DMS, J10 PRECHARGE_CONTACTOR, J11 STO OUT, J13 POWER, J2 ESTOP CONTROLLER, J3 ESTOP EXTERNAL, J4 FENCE, J5 TEACH SWITCH, J6 BRAKES, J7 INPUTS, J8 ISO_CONTACTOR, J9 MAIN_CONTACTOR, K1 Relay_DPDT, K10 Relay_DPDT, K11 Relay_DPDT, K12 Relay_DPDT, K13 Relay_DPDT, K14 Relay_DPDT, K15 Relay_DPDT, K16 Relay_DPDT, K2 Relay_DPDT, K3 Relay_DPDT, K4 Relay_DPDT, K5 Relay_DPDT, K6 Relay_DPDT, K7 Relay_DPDT, K8 Relay_DPDT, K9 Relay_DPDT, U1 140357145400, U10 140357145400, U11 140357145400, U12 140357145400, U13 140357145400, U14 140357145400, U15 140357145400, U16 140357145400, U17 140357145400, U18 ULN2003, U19 74HC165, U2 140357145400, U20 74HC165, U21 74HC165, U22 74HC165, U23 140357145400, U24 140357145400, U25 140357145400, U26 140357145400, U27 140357145400, U28 140357145400, U29 140357145400, U3 140357145400, U30 140357145400, U31 140357145400, U32 140357145400, U33 140357145400, U34 140357145400, U35 140357145400, U36 140357145400, U37 140357145400, U4 140357145400, U41 74HC595, U42 74HC595, U5 ULN2003, U6 140357145400, U7 140357145400, U8 140357145400, U9 140357145400

Commit message: add files
Parts:
- removed the R1 at (616.5, 42.2)
- removed the R10 at (640.3, 45.7)
- removed R100, R101, R96, R97, R98, R99: 9.1k, Resistor_SMD:R_0805_2012Metric
- removed the R11 at (640.3, 49.0)
- removed the R12 at (640.3, 52.3)
- removed the R13 at (640.3, 55.6)
- removed the R14 at (645.9, 42.4)
- removed the R15 at (645.9, 45.7)
- removed the R17 at (645.9, 49.0)
- removed the R18 at (645.9, 52.3)
- removed the R19 at (645.9, 55.6)
- removed the R2 at (616.5, 45.1)
- removed the R25 at (616.5, 51.0)
- removed the R27 at (616.5, 54.0)
- removed the R29 at (616.5, 56.9)
- removed the R3 at (616.5, 48.1)
- removed the R39 at (616.5, 59.9)
- removed the R4 at (634.7, 42.4)
- removed the R42 at (616.5, 62.8)
- removed the R43 at (616.5, 65.8)
- removed the R44 at (620.9, 42.2)
- removed the R45 at (620.9, 45.1)
- removed the R46 at (620.9, 48.1)
- removed the R47 at (620.9, 51.0)
- removed the R48 at (620.9, 54.0)
- removed the R49 at (620.9, 56.9)
- removed the R5 at (634.7, 45.7)
- removed the R50 at (620.9, 59.9)
- removed the R51 at (620.9, 62.8)
- removed the R52 at (620.9, 65.8)
- removed the R53 at (625.3, 42.2)
- removed the R54 at (625.3, 45.1)
- removed the R55 at (625.3, 48.1)
- removed the R56 at (625.3, 51.0)
- removed the R57 at (625.3, 54.0)
- removed the R58 at (625.3, 56.9)
- removed the R59 at (625.3, 59.9)
- removed the R6 at (634.7, 49.0)
- removed the R60 at (625.3, 62.8)
- removed the R61 at (625.3, 65.8)
- removed the R62 at (629.7, 42.2)
- removed the R7 at (634.7, 52.3)
- removed the R8 at (634.7, 55.6)
- removed the R9 at (640.3, 42.4)
- J1, J5: footprint footprints:2x03_P3.5_KF2EDGSR -> footprints:DORABO DB141V-2.54-6P-GN
- J10, J11, J13, J2, J3, J4, J8, J9: footprint footprints:2x02_P3.5_KF2EDGSR -> footprints:DORABO DB141V-2.54-4P-GN
- J6, J7: footprint footprints:2x06_P3.5_KF2EDGSR -> footprints:DORABO DB141V-2.54-12P-GN
- R16: value 33k -> 220k; footprint Resistor_SMD:R_1206_3216Metric -> Resistor_SMD:R_0805_2012Metric
- R20, R21, R22, R23: value 9.1k -> 220k
- R24, R26, R28, R30, R31, R32, R40, R41: value 9.1k -> 2.2k
- R63, R64, R65, R66, R67, R68, R69, R70, R71, R72, R73, R74, R75, R76, R77, R78, R79, R80, R81, R82, R83, R84, R85, R86, R87, R88, R89, R90, R91, R92, R93, R94: value 1.5k -> 220k
- moved J3 102.4 mm to (540.7, 136.5)
Connections:
- D17 pad 2: Net-(D17-A) -> ISO_CONTACTOR_RETURN
- D18 pad 2: Net-(D18-A) -> MAIN_CONTACTOR_RETURN
- D19 pad 2: Net-(D19-A) -> PRECHARGE_CONTACTOR_RETURN
- U15 pad 2: Net-(D17-A) -> ISO_CONTACTOR_RETURN
- U16 pad 2: Net-(D18-A) -> MAIN_CONTACTOR_RETURN
- U17 pad 2: Net-(D19-A) -> PRECHARGE_CONTACTOR_RETURN
- U2 pad 1: Net-(R2-Pad2) -> Net-(R2-Pad1)
- U3 pad 1: Net-(R100-Pad2) -> Net-(R3-Pad1)
